Commit message: Updated simulation launch and plugins

File: src/field_description/urdf/track_example.urdf (robot description, URDF)
Before this commit: robot track_base, 29 links, 28 joints
Links:
- added link zed_link_1, mass 1.2081073109310216; collision mesh filename=package://field_description/meshes/r_bot/zed_link_1.stl scale=0.001 0.001 0.001; visual mesh filename=package://field_description/meshes/r_bot/zed_link_1.stl scale=0.001 0.001 0.001
- added link zed_optical_frame
Joints:
- added joint zed_joint: type fixed, parent base_link, child zed_link_1, origin xyz=0.1 0.05 0.5 rpy=0 0 0
- added joint zed_optical_joint: type fixed, parent zed_link_1, child zed_optical_frame, origin xyz=0 0 0 rpy=-1.5708 0 -1.5708
