Commit message: Add the r2_bringup package

File: src/arm_description/urdf/spear_arm.urdf (robot description, URDF)
Before this commit: robot spear_arm, 9 links, 8 joints
Joints:
- joint base_camera_joint: origin xyz=-0.15 0.15 0.18 rpy=0 0 0 -> xyz=-0.15 0.22 0.18 rpy=0 0 0

File: src/field_description/urdf/r2_base.urdf (robot description, URDF)
Before this commit: robot r2_base, 8 links, 7 joints
Joints:
- joint base_camera_joint: origin xyz=0.2 0 0.28 rpy=0 0 0 -> xyz=0.25 0 0.48 rpy=0 0 0
- joint lidar_joint: origin xyz=0.1 0 0 rpy=0 0 0 -> xyz=0 0 0.03 rpy=3.14 0 0

File: src/field_description/urdf/r_bot.urdf (robot description, URDF)
Before this commit: robot r_bot_wheel, 9 links, 8 joints
Joints:
- joint zed_joint: origin xyz=-0.167758 -0.000778 0.7 rpy=0 0.255 0 -> xyz=-0.167758 -0.000778 0.5 rpy=0 0.255 0
