Commit message: add the robotic arm for moveit2

File: src/kfs_robotic_arm_config/config/arm.ros2_control.xacro (robot description, xacro)
@@ -8,20 +8,20 @@
                 <plugin>mock_components/GenericSystem</plugin>
             </hardware>
-            <joint name="joint_1">
+            <joint name="arm_base_joint">
                 <command_interface name="position"/>
                 <state_interface name="position">
-                  <param name="initial_value">${initial_positions['joint_1']}</param>
+                  <param name="initial_value">${initial_positions['arm_base_joint']}</param>
                 </state_interface>
             </joint>
-            <joint name="joint_2">
+            <joint name="arm_link_joint">
                 <command_interface name="position"/>
                 <state_interface name="position">
-                  <param name="initial_value">${initial_positions['joint_2']}</param>
+                  <param name="initial_value">${initial_positions['arm_link_joint']}</param>
                 </state_interface>
             </joint>
-            <joint name="joint_3">
+            <joint name="gripper_base_joint">
                 <command_interface name="position"/>
                 <state_interface name="position">
-                  <param name="initial_value">${initial_positions['joint_3']}</param>
+                  <param name="initial_value">${initial_positions['gripper_base_joint']}</param>
                 </state_interface>
             </joint>

File: src/kfs_robotic_arm_config/config/arm.urdf.xacro (robot description, xacro)
@@ -3,5 +3,5 @@
     <xacro:arg name="initial_positions_file" default="initial_positions.yaml" />
     <!-- Import arm urdf file -->
-    <xacro:include filename="$(find field_description)/urdf/arm.urdf" />
+    <xacro:include filename="$(find field_description)/urdf/robotic_arm.urdf" />
     <!-- Import control_xacro -->
     <xacro:include filename="arm.ros2_control.xacro" />
